File: MCU-Datalogger.kicad_pcb (KiCad board)
At the start: 2 copper layers, 51.1 x 30 mm, 29 parts, among them J1 Conn_01x04_Pin, J2 Conn_01x04_Pin, J3 Conn_01x09_Pin, J4 Conn_02x03_Odd_Even, U1 24LC1025, U2 24LC1025, U3 DS1337S_, U4 ATMEGA328P-AU, Y1 32.768 KHz, Y2 16 MHz

Commit message: update models
Parts:
- moved H2 0.80 mm to (125.9, 93.9)
- moved H3 0.30 mm to (171.1, 92.4), turned to 90 degrees
- turned H4 to 90 degrees
Changed lines of the file:
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@@
 	(footprint "MountingHole:MountingHole_2.1mm"
 		(layer "F.Cu")
-		(at 170.8 92.4)
+		(at 171.1 92.4 90)
 		(descr "Mounting Hole 2.1mm, no annular")
 		(tags "mounting hole 2.1mm no annular")
 		(property "Reference" "H3"
-			(at 0 -3.2 0)
+			(at 0 -3.2 90)
 			(layer "F.SilkS")
 			(effects
@@
 		)
 		(property "Value" "MountingHole"
-			(at 0 3.2 0)
+			(at 0 3.2 90)
 			(layer "F.Fab")
 			(effects
@@
 		)
 		(property "Datasheet" ""
-			(at 0 0 0)
+			(at 0 0 90)
 			(unlocked yes)
 			(layer "F.Fab")
@@
 		)
 		(property "Description" "Mounting Hole without connection"
-			(at 0 0 0)
+			(at 0 0 90)
 			(unlocked yes)
 			(layer "F.Fab")
@@
 		)
 		(fp_text user "${REFERENCE}"
-			(at 0 0 0)
+			(at 0 0 90)
 			(layer "F.Fab")
 			(effects
@@
 		)
 		(pad "" np_thru_hole circle
-			(at 0 0)
+			(at 0 0 90)
 			(size 2.1 2.1)
 			(drill 2.1)
@@
 	(footprint "MountingHole:MountingHole_2.1mm"
 		(layer "F.Cu")
-		(at 125.9 93.1)
+		(at 125.9 93.9)
 		(descr "Mounting Hole 2.1mm, no annular")
 		(tags "mounting hole 2.1mm no annular")
@@
 		)
 		(embedded_fonts no)
+		(model "${KIPRJMOD}/Libraries/ATMEGA328P-AU/ATMEGA328P-AU.step"
+			(offset
+				(xyz 0 0 0)
+			)
+			(scale
+				(xyz 1 1 1)
+			)
+			(rotate
+				(xyz -90 -0 -0)
+			)
+		)
 	)
 	(footprint "Crystal:Crystal_SMD_5032-2Pin_5.0x3.2mm_HandSoldering"
@@
 		)
 		(embedded_fonts no)
+		(model "${KIPRJMOD}/Libraries/DS1337S_/DS1337S_.step"
+			(offset
+				(xyz 0 0 0)
+			)
+			(scale
+				(xyz 1 1 1)
+			)
+			(rotate
+				(xyz -90 -0 -0)
+			)
+		)
 	)
 	(footprint "Capacitor_SMD:C_0805_2012Metric"
@@
 	(footprint "MountingHole:MountingHole_2.1mm"
 		(layer "F.Cu")
-		(at 171.1 117.5)
+		(at 171.1 117.5 90)
 		(descr "Mounting Hole 2.1mm, no annular")
 		(tags "mounting hole 2.1mm no annular")
 		(property "Reference" "H4"
-			(at 0 -3.2 0)
+			(at 0 -3.2 90)
 			(layer "F.SilkS")
 			(effects
@@
 		)
 		(property "Value" "MountingHole"
-			(at 0 3.2 0)
+			(at 0 3.2 90)
 			(layer "F.Fab")
 			(effects
@@
 		)
 		(property "Datasheet" ""
-			(at 0 0 0)
+			(at 0 0 90)
 			(unlocked yes)
 			(layer "F.Fab")
@@
 		)
 		(property "Description" "Mounting Hole without connection"
-			(at 0 0 0)
+			(at 0 0 90)
 			(unlocked yes)
 			(layer "F.Fab")
@@
 		)
 		(fp_text user "${REFERENCE}"
-			(at 0 0 0)
+			(at 0 0 90)
 			(layer "F.Fab")
 			(effects
@@
 		)
 		(pad "" np_thru_hole circle
-			(at 0 0)
+			(at 0 0 90)
 			(size 2.1 2.1)
 			(drill 2.1)

Commit message: fix bugs
Connections:
- D2 pad 2: /SCL -> /SCK
- J4 pad 3: /SCL -> /SCK
- U4 pad 17: /SCL -> /SCK
Routing:
- net /SCK: track 0.00 -> 36.0 mm, vias 0 -> 3
- net /SCL: track 112.3 -> 87.7 mm, vias 5 -> 2
- net Net-(U4-PB7): track 27.0 -> 49.7 mm
- net Net-(U3-VCC): track 33.2 -> 51.8 mm, vias 0 -> 2
- net /MISO: track 31.3 -> 45.8 mm, vias 2 -> 1
- net /SDA: track 85.0 -> 71.5 mm
- net Net-(D1-K): track 19.2 -> 30.6 mm
- net /RESET: track 29.5 -> 39.9 mm, vias 2 -> 3
- net Net-(U3-SQW/~INT): track 40.2 -> 30.3 mm
- net Net-(U3-~{INTA}): track 39.2 -> 48.5 mm, vias 0 -> 2
- net GND: track 145.9 -> 136.7 mm, vias 4 -> 2
- net /RX: track 23.9 -> 31.8 mm
- net /D7: track 8.91 -> 16.7 mm, vias 0 -> 1
- net /VCC: track 122.4 -> 117.1 mm, vias 1 -> 0
- net /TX: track 35.6 -> 32.0 mm
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