File: MCU-Datalogger.kicad_sch (KiCad schematic)
At the start: 25 parts, among them U1 24LC1025, U2 24LC1025, U3 DS1337S_, U4 ATMEGA328P-AU, Y1 32.768 KHz, Y2 16 MHz

Commit message: fix bugs
Connections:
- net SCL: no longer D2.2 (A), U4.17 (PB5)
- new net SCK: D2.2 (A), U4.17 (PB5)
Other:
- sheet Connectors ports: added SCK; removed none
Changed lines of the file:
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@@
 		)
 	)
-	(label "SCL"
+	(label "SCK"
 		(at 147.32 113.03 180)
 		(effects
@@
 	)
 	(label "SDA"
-		(at 231.14 59.69 180)
+		(at 231.14 54.61 180)
 		(effects
 			(font
@@
 	)
 	(label "SCL"
-		(at 231.14 63.5 180)
+		(at 231.14 58.42 180)
 		(effects
 			(font
@@
 	)
 	(label "MOSI"
-		(at 231.14 83.82 180)
+		(at 231.14 78.74 180)
 		(effects
 			(font
@@
 	)
 	(label "RX"
-		(at 231.14 71.12 180)
+		(at 231.14 66.04 180)
 		(effects
 			(font
@@
 	)
 	(label "MISO"
-		(at 231.14 87.63 180)
+		(at 231.14 82.55 180)
 		(effects
 			(font
@@
 	)
 	(label "TX"
-		(at 231.14 74.93 180)
+		(at 231.14 69.85 180)
+		(effects
+			(font
+				(size 1.27 1.27)
+			)
+			(justify right bottom)
+		)
+	)
+	(label "SCK"
+		(at 231.14 73.66 180)
 		(effects
 			(font
@@
 	)
 	(label "RESET"
-		(at 231.14 91.44 180)
+		(at 231.14 86.36 180)
 		(effects
 			(font
@@
 		)
 		(pin "SDA" bidirectional
-			(at 231.14 59.69 180)
+			(at 231.14 54.61 180)
 			(effects
 				(font
@@
 		)
 		(pin "SCL" passive
-			(at 231.14 63.5 180)
+			(at 231.14 58.42 180)
 			(effects
 				(font
@@
 		)
 		(pin "RX" input
-			(at 231.14 71.12 180)
+			(at 231.14 66.04 180)
 			(effects
 				(font
@@
 		)
 		(pin "TX" output
-			(at 231.14 74.93 180)
+			(at 231.14 69.85 180)
 			(effects
 				(font
@@
 		)
 		(pin "MISO" output
-			(at 231.14 87.63 180)
+			(at 231.14 82.55 180)
 			(effects
 				(font
@@
 		)
 		(pin "RESET" passive
-			(at 231.14 91.44 180)
+			(at 231.14 86.36 180)
 			(effects
 				(font
@@
 		)
 		(pin "MOSI" input
-			(at 231.14 83.82 180)
+			(at 231.14 78.74 180)
+			(effects
+				(font
+					(size 1.27 1.27)
+				)
+				(justify left)
+			)
+		)
+		(pin "SCK" passive
+			(at 231.14 73.66 180)
 			(effects
 				(font
