File: connectors.kicad_sch (KiCad schematic)
At the start: 4 parts, among them J1 Conn_01x04_Pin, J2 Conn_01x04_Pin, J3 Conn_01x09_Pin, J4 Conn_02x03_Odd_Even

Commit message: fix bugs
Connections:
- net SCL: no longer J4.3 (Pin_3)
- new net SCK: J4.3 (Pin_3)
Other:
- moved on the sheet: J1, J2, J3, J4
Changed lines of the file:
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@@
 	(hierarchical_label "D8"
 		(shape bidirectional)
-		(at 77.47 97.79 0)
+		(at 132.08 114.3 0)
 		(effects
 			(font
@@
 	(hierarchical_label "D3"
 		(shape bidirectional)
-		(at 77.47 85.09 0)
+		(at 132.08 101.6 0)
 		(effects
 			(font
@@
 	(hierarchical_label "MOSI"
 		(shape input)
-		(at 109.22 92.71 0)
+		(at 163.83 109.22 0)
 		(effects
 			(font
@@
 	(hierarchical_label "RX"
 		(shape input)
-		(at 102.87 69.85 0)
+		(at 157.48 86.36 0)
 		(effects
 			(font
@@
 	(hierarchical_label "RESET"
 		(shape passive)
-		(at 96.52 95.25 180)
+		(at 151.13 111.76 180)
 		(effects
 			(font
@@
 		)
 	)
-	(hierarchical_label "SCL"
-		(shape passive)
-		(at 96.52 92.71 180)
+	(hierarchical_label "SCK"
+		(shape passive)
+		(at 151.13 109.22 180)
 		(effects
 			(font
@@
 	(hierarchical_label "GND"
 		(shape passive)
-		(at 102.87 64.77 0)
+		(at 157.48 81.28 0)
 		(effects
 			(font
@@
 	(hierarchical_label "TX"
 		(shape output)
-		(at 102.87 72.39 0)
+		(at 157.48 88.9 0)
 		(effects
 			(font
@@
 	(hierarchical_label "MISO"
 		(shape output)
-		(at 96.52 90.17 180)
+		(at 151.13 106.68 180)
 		(effects
 			(font
@@
 	(hierarchical_label "D4"
 		(shape bidirectional)
-		(at 77.47 87.63 0)
+		(at 132.08 104.14 0)
 		(effects
 			(font
@@
 	(hierarchical_label "VCC"
 		(shape passive)
-		(at 77.47 102.87 0)
+		(at 132.08 119.38 0)
 		(effects
 			(font
@@
 	(hierarchical_label "GND"
 		(shape passive)
-		(at 109.22 95.25 0)
+		(at 163.83 111.76 0)
 		(effects
 			(font
@@
 	(hierarchical_label "GND"
 		(shape passive)
-		(at 77.47 100.33 0)
+		(at 132.08 116.84 0)
 		(effects
 			(font
@@
 	(hierarchical_label "D2"
 		(shape bidirectional)
-		(at 77.47 82.55 0)
+		(at 132.08 99.06 0)
 		(effects
 			(font
@@
 	(hierarchical_label "VCC"
 		(shape passive)
-		(at 109.22 90.17 0)
+		(at 163.83 106.68 0)
 		(effects
 			(font
@@
 	(hierarchical_label "SDA"
 		(shape bidirectional)
-		(at 77.47 69.85 0)
+		(at 132.08 86.36 0)
 		(effects
 			(font
@@
 	(hierarchical_label "D5"
 		(shape bidirectional)
-		(at 77.47 90.17 0)
+		(at 132.08 106.68 0)
 		(effects
 			(font
@@
 	(hierarchical_label "SCL"
 		(shape passive)
-		(at 77.47 72.39 0)
+		(at 132.08 88.9 0)
 		(effects
 			(font
@@
 	(hierarchical_label "D7"
 		(shape bidirectional)
-		(at 77.47 95.25 0)
+		(at 132.08 111.76 0)
 		(effects
 			(font
@@
 	(hierarchical_label "GND"
 		(shape passive)
-		(at 77.47 64.77 0)
+		(at 132.08 81.28 0)
 		(effects
 			(font
@@
 	(hierarchical_label "VCC"
 		(shape passive)
-		(at 77.47 67.31 0)
+		(at 132.08 83.82 0)
 		(effects
 			(font
@@
 	(hierarchical_label "D6"
 		(shape bidirectional)
-		(at 77.47 92.71 0)
+		(at 132.08 109.22 0)
 		(effects
 			(font
@@
 	(hierarchical_label "VCC"
 		(shape passive)
-		(at 102.87 67.31 0)
+		(at 157.48 83.82 0)
 		(effects
 			(font
@@
 	(symbol
 		(lib_id "Connector_Generic:Conn_02x03_Odd_Even")
-		(at 101.6 92.71 0)
+		(at 156.21 109.22 0)
 		(unit 1)
 		(exclude_from_sim no)
@@
 		(fields_autoplaced yes)
 		(property "Reference" "J4"
-			(at 102.87 83.82 0)
+			(at 157.48 100.33 0)
 			(effects
 				(font
@@
 		)
 		(property "Value" "Conn_02x03_Odd_Even"
-			(at 102.87 86.36 0)
+			(at 157.48 102.87 0)
 			(effects
 				(font
@@
 		)
 		(property "Footprint" "Connector_PinHeader_2.54mm:PinHeader_2x03_P2.54mm_Vertical"
-			(at 101.6 92.71 0)
+			(at 156.21 109.22 0)
 			(effects
 				(font
@@
 		)
 		(property "Datasheet" "~"
-			(at 101.6 92.71 0)
+			(at 156.21 109.22 0)
 			(effects
 				(font
@@
 		)
 		(property "Description" "Generic connector, double row, 02x03, odd/even pin numbering scheme (row 1 odd numbers, row 2 even numbers), script generated (kicad-library-utils/schlib/autogen/connector/)"
-			(at 101.6 92.71 0)
+			(at 156.21 109.22 0)
 			(effects
 				(font
@@
 	(symbol
 		(lib_id "Connector:Conn_01x04_Pin")
-		(at 97.79 67.31 0)
+		(at 152.4 83.82 0)
 		(unit 1)
 		(exclude_from_sim no)
@@
 		(fields_autoplaced yes)
 		(property "Reference" "J2"
-			(at 98.425 59.69 0)
+			(at 153.035 76.2 0)
 			(effects
 				(font
@@
 		)
 		(property "Value" "Conn_01x04_Pin"
-			(at 98.425 62.23 0)
+			(at 153.035 78.74 0)
 			(effects
 				(font
@@
 		)
 		(property "Footprint" "Connector_PinHeader_2.54mm:PinHeader_1x04_P2.54mm_Vertical"
-			(at 97.79 67.31 0)
+			(at 152.4 83.82 0)
 			(effects
 				(font
@@
 		)
 		(property "Datasheet" "~"
-			(at 97.79 67.31 0)
+			(at 152.4 83.82 0)
 			(effects
 				(font
@@
 		)
 		(property "Description" "Generic connector, single row, 01x04, script generated"
-			(at 97.79 67.31 0)
+			(at 152.4 83.82 0)
 			(effects
 				(font
@@
 	(symbol
 		(lib_id "Connector:Conn_01x04_Pin")
-		(at 72.39 67.31 0)
+		(at 127 83.82 0)
 		(unit 1)
 		(exclude_from_sim no)
@@
 		(fields_autoplaced yes)
 		(property "Reference" "J1"
-			(at 73.025 59.69 0)
+			(at 127.635 76.2 0)
 			(effects
 				(font
@@
 		)
 		(property "Value" "Conn_01x04_Pin"
-			(at 73.025 62.23 0)
+			(at 127.635 78.74 0)
 			(effects
 				(font
@@
 		)
 		(property "Footprint" "Connector_PinHeader_2.54mm:PinHeader_1x04_P2.54mm_Vertical"
-			(at 72.39 67.31 0)
+			(at 127 83.82 0)
 			(effects
 				(font
@@
 		)
 		(property "Datasheet" "~"
-			(at 72.39 67.31 0)
+			(at 127 83.82 0)
 			(effects
 				(font
@@
 		)
 		(property "Description" "Generic connector, single row, 01x04, script generated"
-			(at 72.39 67.31 0)
+			(at 127 83.82 0)
 			(effects
 				(font
@@
 	(symbol
 		(lib_id "Connector:Conn_01x09_Pin")
-		(at 72.39 92.71 0)
+		(at 127 109.22 0)
 		(unit 1)
 		(exclude_from_sim no)
@@
 		(fields_autoplaced yes)
 		(property "Reference" "J3"
-			(at 73.025 77.47 0)
+			(at 127.635 93.98 0)
 			(effects
 				(font
@@
 		)
 		(property "Value" "Conn_01x09_Pin"
-			(at 73.025 80.01 0)
+			(at 127.635 96.52 0)
 			(effects
 				(font
@@
 		)
 		(property "Footprint" "Connector_PinHeader_2.54mm:PinHeader_1x09_P2.54mm_Vertical"
-			(at 72.39 92.71 0)
+			(at 127 109.22 0)
 			(effects
 				(font
@@
 		)
 		(property "Datasheet" "~"
-			(at 72.39 92.71 0)
+			(at 127 109.22 0)
 			(effects
 				(font
@@
 		)
 		(property "Description" "Generic connector, single row, 01x09, script generated"
-			(at 72.39 92.71 0)
-			(effects
-				(font
+			(at 127 109.22 0)
+			(effects
+				(font
